File: kicad/ts/mux.kicad_sch (KiCad schematic)
At the start: 5 parts, among them X0 74LS157, X1 74LS153, X2 74LS153, X3 74LS153, X4 74LS153

Commit message: update footprints
Parts:
- X0: footprint (none) -> Package_DIP:DIP-16_W7.62mm
Changed lines of the file:
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@@
 			)
 		)
-		(property "Footprint" ""
+		(property "Footprint" "Package_DIP:DIP-16_W7.62mm"
 			(at 57.15 57.785 0)
 			(effects
