File: kicad/ts/z80cpu.kicad_sch (KiCad schematic)
At the start: 20 parts, among them M8 27C128, SW1 SW_SPDT_312

Commit message: update footprints
Parts:
- G3, TS1: footprint (none) -> Package_DIP:DIP-14_W7.62mm
- Z1: footprint (none) -> Package_DIP:DIP-40_W15.24mm
Changed lines of the file:
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@@
 			)
 		)
-		(property "Footprint" ""
+		(property "Footprint" "Package_DIP:DIP-14_W7.62mm"
 			(at 69.215 72.39 0)
 			(effects
@@
 			)
 		)
-		(property "Footprint" ""
+		(property "Footprint" "Package_DIP:DIP-14_W7.62mm"
 			(at 50.8 60.96 0)
 			(effects
@@
 			)
 		)
-		(property "Footprint" ""
+		(property "Footprint" "Package_DIP:DIP-14_W7.62mm"
 			(at 69.215 60.96 0)
 			(effects
@@
 			)
 		)
-		(property "Footprint" ""
+		(property "Footprint" "Package_DIP:DIP-40_W15.24mm"
 			(at 137.795 86.995 0)
 			(effects
@@
 			)
 		)
-		(property "Footprint" ""
+		(property "Footprint" "Package_DIP:DIP-14_W7.62mm"
 			(at 88.9 66.675 0)
 			(effects

Commit message: Schemativ corrections, work started on pcb
Parts:
- SW1: footprint Button_Switch_THT:SW_XKB_DM1-16UC-1 -> Cobra_original:Reset_Switch
Changed lines of the file:
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@@
 			)
 		)
-		(property "Footprint" "Button_Switch_THT:SW_XKB_DM1-16UC-1"
+		(property "Footprint" "Cobra_original:Reset_Switch"
 			(at 37.465 92.075 0)
 			(effects

Commit message: More pcb work
Parts:
- SW1: footprint Cobra_original:Reset_Switch -> Cobra_original:Reset_Switch3p
Changed lines of the file:
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@@
 			)
 		)
-		(property "Footprint" "Cobra_original:Reset_Switch"
+		(property "Footprint" "Cobra_original:Reset_Switch3p"
 			(at 37.465 92.075 0)
 			(effects
