File: kicad/ts/IO.kicad_sch (KiCad schematic)
At the start: 32 parts, among them J3 AudioJack3

Commit message: update footprints
Parts:
- B1, F5: footprint (none) -> Package_DIP:DIP-20_W7.62mm
Changed lines of the file:
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@@
 			)
 		)
-		(property "Footprint" ""
+		(property "Footprint" "Package_DIP:DIP-20_W7.62mm"
 			(at 139.7 54.61 0)
 			(effects
@@
 			)
 		)
-		(property "Footprint" ""
+		(property "Footprint" "Package_DIP:DIP-20_W7.62mm"
 			(at 59.055 54.61 0)
 			(effects

Commit message: Schemativ corrections, work started on pcb
Parts:
- J3, JTI1, JTO1: footprint (none) -> Connector_Audio:Jack_3.5mm_CUI_SJ1-3533NG_Horizontal_CircularHoles
Changed lines of the file:
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@@
 			)
 		)
-		(property "Footprint" ""
+		(property "Footprint" "Connector_Audio:Jack_3.5mm_CUI_SJ1-3533NG_Horizontal_CircularHoles"
 			(at 70.485 197.485 0)
 			(effects
@@
 			)
 		)
-		(property "Footprint" ""
+		(property "Footprint" "Connector_Audio:Jack_3.5mm_CUI_SJ1-3533NG_Horizontal_CircularHoles"
 			(at 152.4 194.31 0)
 			(effects
@@
 			)
 		)
-		(property "Footprint" ""
+		(property "Footprint" "Connector_Audio:Jack_3.5mm_CUI_SJ1-3533NG_Horizontal_CircularHoles"
 			(at 125.095 119.38 0)
 			(effects

Commit message: More pcb work
Parts:
- JKB1: footprint (none) -> Connector_PinHeader_2.54mm:PinHeader_2x10_P2.54mm_Vertical
Changed lines of the file:
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@@
 			)
 		)
-		(property "Footprint" ""
+		(property "Footprint" "Connector_PinHeader_2.54mm:PinHeader_2x10_P2.54mm_Vertical"
 			(at 95.25 133.35 0)
 			(effects

Commit message: Schematic corrections, more traces to pcb, update to DIN 3x32 connector footprint
Parts:
- J3, JTI1, JTO1: footprint Connector_Audio:Jack_3.5mm_CUI_SJ1-3533NG_Horizontal_CircularHoles -> Connector_Audio:Jack_3.5mm_CUI_SJ1-3533NG_Horizontal
Changed lines of the file:
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@@
 			)
 		)
-		(property "Footprint" "Connector_Audio:Jack_3.5mm_CUI_SJ1-3533NG_Horizontal_CircularHoles"
+		(property "Footprint" "Connector_Audio:Jack_3.5mm_CUI_SJ1-3533NG_Horizontal"
 			(at 70.485 197.485 0)
 			(effects
@@
 			)
 		)
-		(property "Footprint" "Connector_Audio:Jack_3.5mm_CUI_SJ1-3533NG_Horizontal_CircularHoles"
+		(property "Footprint" "Connector_Audio:Jack_3.5mm_CUI_SJ1-3533NG_Horizontal"
 			(at 152.4 194.31 0)
 			(effects
@@
 			)
 		)
-		(property "Footprint" "Connector_Audio:Jack_3.5mm_CUI_SJ1-3533NG_Horizontal_CircularHoles"
+		(property "Footprint" "Connector_Audio:Jack_3.5mm_CUI_SJ1-3533NG_Horizontal"
 			(at 125.095 119.38 0)
 			(effects

Commit message: 4164 footprint corrected, more pcb traces
Parts:
- CAO1: footprint (none) -> Capacitor_THT:CP_Radial_D5.0mm_P2.50mm
Changed lines of the file:
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@@
 			)
 		)
-		(property "Footprint" ""
+		(property "Footprint" "Capacitor_THT:CP_Radial_D5.0mm_P2.50mm"
 			(at 121.92 109.855 0)
 			(effects

Commit message: minor updates
Connections:
- net GNDD: now also DTO0.2 (A), DTO1.1 (K); no longer DTO0.1 (K), DTO1.2 (A)
- net at RQ3.2, RTO1.1: now also DTO0.1 (K), DTO1.2 (A); no longer DTO0.2 (A), DTO1.1 (K)
Other:
- moved on the sheet: DTO0, DTO1
Changed lines of the file:
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@@
 	(symbol
 		(lib_id "Diode:1N4148")
-		(at 129.54 201.93 270)
+		(at 129.54 201.93 90)
 		(unit 1)
 		(exclude_from_sim no)
@@
 		(dnp no)
 		(property "Reference" "DTO1"
-			(at 133.985 201.295 90)
+			(at 133.985 202.565 90)
 			(effects
 				(font
@@
 		)
 		(property "Value" "1N4148"
-			(at 135.255 203.2 90)
+			(at 135.255 200.66 90)
 			(effects
 				(font
@@
 	(symbol
 		(lib_id "Diode:1N4148")
-		(at 125.73 201.93 90)
+		(at 125.73 201.93 270)
 		(unit 1)
 		(exclude_from_sim no)
@@
 		(dnp no)
 		(property "Reference" "DTO0"
-			(at 121.285 201.295 90)
+			(at 121.285 202.565 90)
 			(effects
 				(font
@@
 		)
 		(property "Value" "1N4148"
-			(at 120.015 203.2 90)
-			(effects
-				(font
+			(at 120.015 200.66 90)
+			(effects
+				(font
